File: hardware/prideocarina/prideocarina.kicad_sch (KiCad schematic)
At the start: 23 parts, among them SW1 SW_Push, SW2 SW_Push, SW3 SW_Push, SW4 SW_Push, SW5 SW_Push, SW6 SW_Push, SW7 SW_Push

Commit message: update schematics
Parts:
- added SW8: SW_Push, symbol Switch:SW_Push
- added TP1: TestPoint, MountingHole:MountingHole_8.4mm_M8_Pad_Via, symbol Connector:TestPoint
- added U1: 74HC138, Package_DIP:DIP-16_W7.62mm, symbol 74xx:74HC138
Connections:
- net +3.3V: now reaches A1.17 (3V3)
- net +5V: now reaches A1.27 (+5V)
- net +5V: now also SW1.1, SW2.1, SW3.1, SW4.1, SW5.1, SW6.1, SW7.1, U1.16 (VCC), U1.6 (E2)
- net RESET: now reaches A1.28 (~{RESET})
- net RESET: now also A1.3 (~{RESET}), SW8.2
- net GND: now reaches A1.29 (GND), A1.4 (GND)
- net GND: now also BT1.2 (-), R1.2, SW8.1, U1.4 (~{E0}), U1.5 (~{E1}), U1.8 (GND)
- net +9V: now reaches A1.30 (VIN)
- net +9V: now also BT1.1 (+)
- net R: now reaches D6.1 (RA)
- net R: now also D1.1 (RA), D2.1 (RA), D3.1 (RA), D4.1 (RA), D5.1 (RA)
- net at D6.2 (K): now also R7.1
- net G: now reaches D6.3 (GA)
- net G: now also D1.3 (GA), D2.3 (GA), D3.3 (GA), D4.3 (GA), D5.3 (GA)
- net B: now reaches D6.4 (BA)
- net B: now also D1.4 (BA), D2.4 (BA), D3.4 (BA), D4.4 (BA), D5.4 (BA)
- net at D2.2 (K): now also R3.1
- net at R4.1: now also D3.2 (K)
- net LED2: now reaches R4.2
- net LED2: now also U1.13 (~{Y2})
- net at D5.2 (K): now also R6.1
- net at R2.1: now also D1.2 (K)
- net LED0: now reaches R2.2
- net LED0: now also U1.15 (~{Y0})
- net LED4: now reaches R6.2
- net LED4: now also U1.11 (~{Y4})
- net SW5: now reaches SW5.2
- net SW6: now reaches SW6.2
- net SW6: now also SW7.2
- net at R1.1: now also LS1.2
- net SPEAK: now reaches LS1.1
- net at D4.2 (K): now also R5.1
- net LED5: now reaches R7.2
- net LED5: now also U1.10 (~{Y5})
- net LED3: now reaches R5.2
- net LED3: now also U1.12 (~{Y3})
- net LED1: now reaches R3.2
- net LED1: now also U1.14 (~{Y1})
- net SW4: now reaches SW4.2
- net SW3: now reaches SW3.2
- net SW2: now reaches SW2.2
- net SW1: now reaches SW1.2
- new net CAP_TOUCH: TP1.1
- new net LEDCTL0: U1.1 (A0)
- new net LEDCTL1: U1.2 (A1)
- new net LEDCTL2: U1.3 (A2)
Other:
- moved on the sheet: D1, D2, D3, D4, D5, D6, R2, R3, R4, R5, R6, R7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

Commit message: finished shema
Parts:
- removed SW7: SW_Push, symbol Switch:SW_Push
- added R8: R_US, Resistor_THT:R_Axial_DIN0309_L9.0mm_D3.2mm_P12.70mm_Horizontal, symbol Device:R_US
Connections:
- net CAP_TOUCH is gone; now on net CAP_TOUCH_RECEIVE: TP1.1
- net B: now also A1.10 (D7)
- net G: now also A1.9 (D6)
- net LEDCTL0: now also A1.5 (D2)
- net LEDCTL1: now also A1.6 (D3)
- net LEDCTL2: now also A1.7 (D4)
- net R: now also A1.8 (D5)
- net SPEAK: now also A1.11 (D8)
- net SW1: now also A1.19 (A0)
- net SW2: now also A1.20 (A1)
- net SW3: now also A1.21 (A2)
- net SW4: now also A1.22 (A3)
- net SW5: now also A1.23 (SDA/A4)
- net SW6: now also A1.24 (SCL/A5)
- net CAP_TOUCH_SEND: now reaches A1.12 (D9)
- net CAP_TOUCH_SEND: now also R8.2
- net CAP_TOUCH_RECEIVE: now reaches A1.13 (D10)
- net CAP_TOUCH_RECEIVE: now also R8.1
