File: hardware/prideocarina/prideocarina.kicad_pcb (KiCad board)
At the start: 2 copper layers, 26 parts, among them SW1 SW_Push, SW2 SW_Push, SW3 SW_Push, SW4 SW_Push, SW5 SW_Push, SW6 SW_Push, SW8 SW_Push, U1 74HC138

Commit message: add more description
Parts:
- added REF**: MountingHole_8.4mm_M8_Pad, MountingHole:MountingHole_8.4mm_M8_Pad, F.Cu at (140.5, 124.5)
- moved R8 120.9 mm to (74.3, 92.0)
- moved TP1 117.1 mm to (67.7, 59.9)
- moved R2 78.4 mm to (122.5, 113.2)
- moved R3 78.4 mm to (117.8, 113.2)
- moved R4 78.4 mm to (113.0, 113.2)
- moved D3 78.0 mm to (109.5, 105.0), turned to 0 degrees
- moved D2 76.1 mm to (124.0, 105.0), turned to 0 degrees
- moved D1 74.5 mm to (141.0, 105.0), turned to 0 degrees
- moved R5 69.6 mm to (74.2, 78.0), turned to 0 degrees
- moved R6 68.8 mm to (74.2, 82.8), turned to 0 degrees
- moved R7 68.6 mm to (74.2, 87.5), turned to 0 degrees
- moved D4 60.8 mm to (94.5, 82.7)
- moved A1 54.2 mm to (52.5, 110.8)
- moved BT1 52.9 mm to (94.5, 97.0)
- moved SW4 48.4 mm to (142.2, 147.2), turned to 180 degrees
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Routing:
- net +5V: track 0.00 -> 205.8 mm
- net R: track 0.00 -> 128.1 mm
- net CAP_TOUCH_RECEIVE: track 0.00 -> 124.9 mm
- net GND: track 0.00 -> 114.8 mm
- net SW4: track 0.00 -> 93.2 mm
- net SW5: track 0.00 -> 76.3 mm
- net SW6: track 0.00 -> 62.5 mm
- net SPEAK: track 0.00 -> 60.5 mm
- net LEDCTL0: track 0.00 -> 49.8 mm
- net LEDCTL1: track 0.00 -> 46.0 mm
- net Net-(D4-K): track 0.00 -> 42.6 mm
- net Net-(D5-K): track 0.00 -> 40.5 mm
- net Net-(D6-K): track 0.00 -> 39.6 mm
- net LED3: track 0.00 -> 36.4 mm
- net LEDCTL2: track 0.00 -> 35.6 mm
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Other:
- board outline added: 100 x 100 mm
